Commit message: Add Gazebo simulation and tune Nav2 navigation

File: robot_ws/src/robot_model/urdf/diffbot.urdf.xacro (robot description, xacro)
@@ -8,4 +8,5 @@
   <xacro:arg name="imu_frame" default="gyro_link"/>
   <xacro:arg name="laser_frame" default="laser"/>
+  <xacro:arg name="use_sim" default="false"/>
   <!-- Yaw (radians) of the LiDAR scan frame relative to base_link forward
        (+X). The RPLidar driver already reports angle zero along the sensor's
@@ -67,7 +68,6 @@
   </link>
   <!-- ============================================================
-       Wheels (visual only - fixed joints; the real/simulated drive
-       external odometry EKF is responsible for publishing odom -> base_link,
-       so no joint_state_publisher is required for navigation)
+       Wheels. Hardware mode keeps them fixed because the base driver does
+       not publish joint states. Simulation mode uses continuous joints.
        ============================================================ -->
   <xacro:macro name="wheel" params="prefix reflect">
@@ -92,9 +92,25 @@
       </inertial>
     </link>
-    <joint name="${prefix}_wheel_joint" type="fixed">
-      <parent link="${base_frame}"/>
-      <child link="${prefix}_wheel_link"/>
-      <origin xyz="0 ${reflect * wheel_separation/2} ${-wheel_radius}" rpy="0 0 0"/>
-    </joint>
+    <xacro:unless value="$(arg use_sim)">
+      <joint name="${prefix}_wheel_joint" type="fixed">
+        <parent link="${base_frame}"/>
+        <child link="${prefix}_wheel_link"/>
+        <origin xyz="0 ${reflect * wheel_separation/2} ${-wheel_radius}" rpy="0 0 0"/>
+      </joint>
+    </xacro:unless>
+    <xacro:if value="$(arg use_sim)">
+      <joint name="${prefix}_wheel_joint" type="continuous">
+        <parent link="${base_frame}"/>
+        <child link="${prefix}_wheel_link"/>
+        <origin xyz="0 ${reflect * wheel_separation/2} ${-wheel_radius}" rpy="0 0 0"/>
+        <!-- Positive joint velocity must roll the wheel toward base +X. -->
+        <axis xyz="0 1 0"/>
+        <dynamics damping="0.02" friction="0.0"/>
+      </joint>
+      <gazebo reference="${prefix}_wheel_link">
+        <mu1>1.0</mu1>
+        <mu2>1.0</mu2>
+      </gazebo>
+    </xacro:if>
   </xacro:macro>
   <xacro:wheel prefix="left" reflect="1"/>
@@ -119,9 +135,26 @@
     </inertial>
   </link>
-  <joint name="caster_wheel_joint" type="fixed">
-    <parent link="${base_frame}"/>
-    <child link="caster_wheel_link"/>
-    <origin xyz="${-chassis_length/2 + caster_radius} 0 ${-wheel_radius + caster_radius}" rpy="0 0 0"/>
-  </joint>
+  <xacro:unless value="$(arg use_sim)">
+    <joint name="caster_wheel_joint" type="fixed">
+      <parent link="${base_frame}"/>
+      <child link="caster_wheel_link"/>
+      <origin xyz="${-chassis_length/2 + caster_radius} 0 ${-wheel_radius + caster_radius}" rpy="0 0 0"/>
+    </joint>
+  </xacro:unless>
+  <xacro:if value="$(arg use_sim)">
+    <joint name="caster_wheel_joint" type="fixed">
+      <parent link="${base_frame}"/>
+      <child link="caster_wheel_link"/>
+      <origin xyz="${-chassis_length/2 + caster_radius} 0 ${-2*wheel_radius + caster_radius}" rpy="0 0 0"/>
+    </joint>
+  </xacro:if>
+  <xacro:if value="$(arg use_sim)">
+    <!-- The display-only hardware caster is above the wheel contact plane.
+         Simulation lowers the full caster link to support the base. -->
+    <gazebo reference="caster_wheel_link">
+      <mu1>0.001</mu1>
+      <mu2>0.001</mu2>
+    </gazebo>
+  </xacro:if>
   <!-- Cartographer requires its tracking-frame origin to be colocated with
        the IMU. Keep that frame FLU, then express the installed H30 FRD axes
@@ -170,3 +203,82 @@
             rpy="${pi} 0 ${-laser_yaw}"/>
   </joint>
+  <xacro:if value="$(arg use_sim)">
+    <gazebo reference="${imu_frame}">
+      <sensor name="imu_sensor" type="imu">
+        <always_on>true</always_on>
+        <update_rate>100</update_rate>
+        <topic>/imu_data_ros</topic>
+        <gz_frame_id>${imu_frame}</gz_frame_id>
+        <imu>
+          <angular_velocity>
+            <x><noise type="gaussian"><mean>0.0</mean><stddev>0.002</stddev></noise></x>
+            <y><noise type="gaussian"><mean>0.0</mean><stddev>0.002</stddev></noise></y>
+            <z><noise type="gaussian"><mean>0.0</mean><stddev>0.002</stddev></noise></z>
+          </angular_velocity>
+          <linear_acceleration>
+            <x><noise type="gaussian"><mean>0.0</mean><stddev>0.02</stddev></noise></x>
+            <y><noise type="gaussian"><mean>0.0</mean><stddev>0.02</stddev></noise></y>
+            <z><noise type="gaussian"><mean>0.0</mean><stddev>0.02</stddev></noise></z>
+          </linear_acceleration>
+        </imu>
+      </sensor>
+    </gazebo>
+    <gazebo reference="${laser_frame}">
+      <sensor name="lidar_sensor" type="gpu_lidar">
+        <always_on>true</always_on>
+        <visualize>true</visualize>
+        <update_rate>10</update_rate>
+        <topic>/scan</topic>
+        <gz_frame_id>${laser_frame}</gz_frame_id>
+        <lidar>
+          <scan>
+            <horizontal>
+              <samples>720</samples>
+              <resolution>1</resolution>
+              <min_angle>-${pi}</min_angle>
+              <max_angle>${pi}</max_angle>
+            </horizontal>
+          </scan>
+          <range>
+            <min>0.15</min>
+            <max>8.0</max>
+            <resolution>0.01</resolution>
+          </range>
+          <noise>
+            <type>gaussian</type>
+            <mean>0.0</mean>
+            <stddev>0.005</stddev>
+          </noise>
+        </lidar>
+      </sensor>
+    </gazebo>
+    <gazebo>
+      <plugin filename="gz-sim-diff-drive-system"
+              name="gz::sim::systems::DiffDrive">
+        <left_joint>left_wheel_joint</left_joint>
+        <right_joint>right_wheel_joint</right_joint>
+        <wheel_separation>${wheel_separation}</wheel_separation>
+        <wheel_radius>${wheel_radius}</wheel_radius>
+        <topic>/cmd_vel</topic>
+        <odom_topic>/odom/raw</odom_topic>
+        <tf_topic>/sim/odom_tf</tf_topic>
+        <frame_id>odom</frame_id>
+        <child_frame_id>${base_frame}</child_frame_id>
+        <odom_publish_frequency>50</odom_publish_frequency>
+        <max_linear_velocity>0.8</max_linear_velocity>
+        <min_linear_velocity>-0.8</min_linear_velocity>
+        <max_angular_velocity>3.0</max_angular_velocity>
+        <min_angular_velocity>-3.0</min_angular_velocity>
+        <max_linear_acceleration>0.8</max_linear_acceleration>
+        <min_linear_acceleration>-0.8</min_linear_acceleration>
+        <max_angular_acceleration>2.0</max_angular_acceleration>
+        <min_angular_acceleration>-2.0</min_angular_acceleration>
+      </plugin>
+      <plugin filename="gz-sim-joint-state-publisher-system"
+              name="gz::sim::systems::JointStatePublisher">
+        <topic>/joint_states</topic>
+        <update_rate>30</update_rate>
+      </plugin>
+    </gazebo>
+  </xacro:if>
 </robot>
