Commit message: Oct 21: Working point to point, fixing cmd_vel and behavior server

File: rb3302_final_proj_code/robot_ws/src/robot_model/urdf/diffbot.urdf.xacro (robot description, xacro)
@@ -19,12 +19,14 @@
   <!-- ============================================================
        Configurable physical dimensions
+       I changed it to the actual dimensions of the robot, originally the length is 0.3 width is 0.25, height is 0.10
        ============================================================ -->
-  <xacro:property name="chassis_length" value="0.30"/>
-  <xacro:property name="chassis_width" value="0.25"/>
-  <xacro:property name="chassis_height" value="0.10"/>
+  <xacro:property name="chassis_length" value="0.17"/>
+  <xacro:property name="chassis_width" value="0.17"/>
+  <xacro:property name="chassis_height" value="0.18"/>
   <xacro:property name="chassis_mass" value="5.0"/>
   <xacro:property name="wheel_radius" value="0.033"/>
   <xacro:property name="wheel_width" value="0.02"/>
-  <xacro:property name="wheel_separation" value="0.288"/>
+  <!-- Changed it to 0.125 from 0.288-->
+  <xacro:property name="wheel_separation" value="0.125"/>
   <xacro:property name="wheel_mass" value="0.5"/>
   <xacro:property name="caster_radius" value="0.015"/>
